File: Feather-M4-Express-Reuse.kicad_pcb (KiCad board)
At the start: 4 copper layers, 88.9 x 50.8 mm, 60 parts, among them J1 JST_SH4, J2 USB_C_Receptacle_USB2.0_16P, J3 JST_SH3, J4 JST_SH3, J5 JST_PH2, J6 Conn_01x12, J7 Conn_01x16, J8 Micro_SD_Card_Det2, Q3 DMP2045U, SW1 KMR2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

Commit message: Latest Revision
Parts:
- removed U7: ATSAMD51J19A-MUT, Adafruit Feather M4 Express:PQFN64-1_Modified
- added C18: 1uF, Capacitor_SMD:C_0603_1608Metric_Pad1.08x0.95mm_HandSolder, F.Cu at (191.7, 106.0)
- added C19: 1uF, Capacitor_SMD:C_0603_1608Metric_Pad1.08x0.95mm_HandSolder, F.Cu at (126.0, 119.3)
- added C20: 1uF, Capacitor_SMD:C_0603_1608Metric_Pad1.08x0.95mm_HandSolder, F.Cu at (130.0, 119.3)
- added U4: TXU0101DCKR, TXU0101DCKR:SC70-6_DCK_TEX-M, F.Cu at (128.0, 122.5)
- added U5: ATSAMD51J19A-MUT, ul_ATSAMD51J19A-MUT:QFN64_9x9MC_MCH-M_Modified, F.Cu at (145.8, 103.4)
- C15: value 1uF -> 10uF; footprint Capacitor_SMD:C_0603_1608Metric_Pad1.08x0.95mm_HandSolder -> Capacitor_SMD:C_0805_2012Metric_Pad1.18x1.45mm_HandSolder
- D4: value MBR120VLSF -> MBR120VLSFT1G; footprint Adafruit Feather M4 Express:SOD-123 -> MBR120VLSFT1G:DIOM3616X98N
- J8: value Micro_SD_Card_Det2 -> 10102166A812A; footprint Connector_Card:microSD_HC_Molex_104031-0811 -> 10102166A812A:AMPHENOL_10102166A812A
- LED1: value WS2812B3535 -> WS2812B
- Q3: footprint Adafruit Feather M4 Express:SOT23-R -> DMP2045U:SOT-23_DIO
- R11, R12, R13: value 100K 1% -> 100K 0.1%
- R7: value 2.2K -> 10K
- U2: footprint Adafruit Feather M4 Express:SOT23-5 -> AP2112K_3_3TRG1:SOT_RG1_DIO
- U3: footprint Adafruit Feather M4 Express:SOT23-5 -> MCP73831T_2ACI_OT:SOT-23-5_MC_MCH-M
- moved TP1 44.2 mm to (124.2, 125.9)
- moved R12 37.2 mm to (171.9, 95.2), turned to 180 degrees
- moved LED1 35.2 mm to (128.0, 126.8)
- moved R13 32.8 mm to (170.1, 93.5), turned to 180 degrees
- moved C17 31.9 mm to (131.9, 126.8), turned to -90 degrees
- moved R4 11.9 mm to (164.6, 120.0)
- moved C12 11.6 mm to (162.6, 120.0)
- moved J4 7.56 mm to (200.7, 122.0), turned to 0 degrees
- moved R15 6.05 mm to (179.2, 89.6)
- moved R2 6.03 mm to (176.8, 89.6)
- moved J3 4.91 mm to (182.8, 121.7)
- moved R10 4.89 mm to (177.5, 122.6)
- moved R6 4.88 mm to (177.5, 119.2)
- moved R1 4.88 mm to (177.5, 120.9)
- moved D3 4.26 mm to (179.2, 84.4)
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Connections:
- net /V_DIV renamed /BATT_VOLT_DIVIDER
- net Net-(U3-PROG) renamed /LIPO_PROG
- C17 pad 1: +3.3V -> VBUS
- D1 pad 1: Net-(D1-K) -> /LIPO_STAT
- D1 pad 2: VBUS -> Net-(D1-A)
- D3 pad 1: GND -> Net-(D3-K)
- D3 pad 2: Net-(D3-A) -> /LIPO_STAT
- J6 pad 2: /EN -> /LDO_ENABLE
- J8 pad 10: unconnected-(J8-DET_A-Pad10) -> GND
- J8 pad 11: GND -> unconnected-(J8-Pad11)
- LED1 pad 1: /D8_NEOPIX -> Net-(LED1-DO)
- LED1 pad 2: +3.3V -> GND
- LED1 pad 3: Net-(LED1-DO) -> /D8_NEOPIX
- LED1 pad 4: GND -> VBUS
- R15 pad 1: Net-(U3-STAT) -> Net-(D3-K)
- R15 pad 2: Net-(D3-A) -> GND
- R2 pad 1: Net-(D1-K) -> VBUS
- R2 pad 2: Net-(U3-STAT) -> Net-(D1-A)
- U1 pad 2: /QSPI_DATA[1] -> /QSPI_DATA_1
- U1 pad 3: /QSPI_DATA[2] -> /QSPI_DATA_2
- U1 pad 5: /QSPI_DATA[0] -> /QSPI_DATA_0
- U1 pad 6: /QSPI_SCK -> /QSPI_CLOCK
- U1 pad 7: /QSPI_DATA[3] -> /QSPI_DATA_3
- U3 pad 1: Net-(U3-STAT) -> /LIPO_STAT
Routing:
- net Net-(U3-STAT): track 58.1 -> 0.00 mm, vias 2 -> 0
- net /LIPO_STAT: track 0.00 -> 57.8 mm, vias 0 -> 2
- net /LDO_ENABLE: track 3.53 -> 53.6 mm
- net /MCU_D8_NEOPIX: track 0.00 -> 47.6 mm, vias 0 -> 4
- net /BATT_VOLT_DIVIDER: track 75.5 -> 36.2 mm
- net VBUS: track 122.4 -> 148.6 mm
- net /D8_NEOPIX: track 19.9 -> 6.13 mm
- net /QSPI_DATA_0: track 0.00 -> 13.1 mm, vias 0 -> 2
- net /QSPI_DATA[0]: track 13.1 -> 0.00 mm, vias 2 -> 0
- net GND: track 120.8 -> 133.9 mm, vias 44 -> 60
- net /QSPI_SCK: track 11.6 -> 0.00 mm, vias 2 -> 0
- net /QSPI_CLOCK: track 0.00 -> 11.6 mm, vias 0 -> 2
- net /MOSI: track 97.1 -> 108.6 mm
- net /QSPI_DATA_2: track 0.00 -> 10.9 mm
- net /QSPI_DATA[2]: track 10.9 -> 0.00 mm
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Other:
- board text added: "*"
- board text added: "0"
- board text added: "0 mils"
- board text added: "0.0091"
- board text added: "0.6 mils"
- board text added: "1"
- board text added: "1.8 mils"
- board text added: "3.3"
- board text added: "3.61"
- board text added: "3.87"
- board text added: "39 mils"
- board text added: "7.87 mils"
- board text added: "B.Cu"
- board text added: "B.Mask"
- board text added: "B.Paste"
- board text added: "B.Silkscreen"
- board text added: "Benjamin Crockett SAMD51 Business Express"
- board text added: "Bottom Silk Screen"
- board text added: "Bottom Solder Mask"
- board text added: "Bottom Solder Paste"
- board text added: "Color"
- board text added: "Dielectric"
- board text added: "Epsilon R"
- board text added: "F.Cu"
- board text added: "F.Mask"
- board text added: "F.Paste"
- board text added: "F.Silkscreen"
- board text added: "FR4 natural"
- board text added: "FR408-HR"
- board text added: "In1.Cu"
- board text added: "In2.Cu"
- board text added: "Layer Name"
- board text added: "Loss Tangent"
- board text added: "Material"
- board text added: "Not specified"
- board text added: "Purple"
- board text added: "TO DO: Add Tear Drops Length match NOR Flash signals. Fix LED 3D Models. Update NeoPixel Footprint and 3D Model. Check SW1 Footprint against datasheet. Fix Solder Stencil openings for the SAMD51."
- board text added: "Thickness (mils)"
- board text added: "Top Silk Screen"
- board text added: "Top Solder Mask"
- board text added: "Top Solder Paste"
- board text added: "Type"
- board text added: "White"
- board text added: "copper"
- board text added: "core"
- board text added: "prepreg"
