File: Feather-M4-Express-Reuse.kicad_sch (KiCad schematic)
At the start: 60 parts, among them J1 JST_SH4, J2 USB_C_Receptacle_USB2.0_16P, J3 JST_SH3, J4 JST_SH3, J5 JST_PH2, J6 Conn_01x12, J7 Conn_01x16, J8 Micro_SD_Card_Det2, Q3 DMP2045U, SW1 KMR2, U1 W25Q128JVSIQ, U2 AP2112-3.3, U3 MCP73831T-2ACI/OT, U7 ATSAMD51J19A-MUT, Y1 32.768 kHz

Commit message: Latest Revision
Parts:
- removed D4: MBR120VLSF, Adafruit Feather M4 Express:SOD-123, symbol Device:D_Schottky
- removed J8: Micro_SD_Card_Det2, Connector_Card:microSD_HC_Molex_104031-0811, symbol Connector:Micro_SD_Card_Det2
- removed U7: ATSAMD51J19A-MUT, Adafruit Feather M4 Express:PQFN64-1_Modified, symbol 2025-09-06_23-45-11:ATSAMD51J19A-MUT
- added C18, C19, C20: 1uF, Capacitor_SMD:C_0603_1608Metric_Pad1.08x0.95mm_HandSolder, symbol Device:C
- added D4: MBR120VLSFT1G, MBR120VLSFT1G:DIOM3616X98N, symbol MBR120VLSFT1G:MBR120VLSFT1G
- added J8: 10102166A812A, 10102166A812A:AMPHENOL_10102166A812A, symbol 10102166A812A:10102166A812A
- added U4: TXU0101DCKR, TXU0101DCKR:SC70-6_DCK_TEX-M, symbol TXU0101DCKR:TXU0101DCKR
- added U5: ATSAMD51J19A-MUT, ul_ATSAMD51J19A-MUT:QFN64_9x9MC_MCH-M_Modified, symbol ATSAMD51J19A-M:ATSAMD51J19A-MUT
- C15: value 1uF -> 10uF; footprint Capacitor_SMD:C_0603_1608Metric_Pad1.08x0.95mm_HandSolder -> Capacitor_SMD:C_0805_2012Metric_Pad1.18x1.45mm_HandSolder
- LED1: value WS2812B3535 -> WS2812B
- Q3: footprint Adafruit Feather M4 Express:SOT23-R -> DMP2045U:SOT-23_DIO
- R11, R12, R13: value 100K 1% -> 100K 0.1%
- R7: value 2.2K -> 10K
- U2: footprint Adafruit Feather M4 Express:SOT23-5 -> AP2112K_3_3TRG1:SOT_RG1_DIO
- U3: footprint Adafruit Feather M4 Express:SOT23-5 -> MCP73831T_2ACI_OT:SOT-23-5_MC_MCH-M
Connections:
- net EN is gone; now on net LDO_ENABLE: J6.2 (Pin_2)
- net +3.3V: now also C18.1, C19.1, J8.4, U4.1 (VCCA), U5.16 (PA07), U5.21 (VDDIO), U5.34 (VDDIO), U5.48 (VDDIO), U5.56 (VDDIO), U5.8 (VDDANA); no longer C17.1, LED1.2 (VDD)
- net A0: now also U5.3 (PA02)
- net A1: now also U5.14 (PA05)
- net A2: now also U5.11 (PB08)
- net A3: now also U5.12 (PB09)
- net A4: now also U5.13 (PA04)
- net A5: now also U5.15 (PA06)
- net AREF: now also U5.4 (PA03)
- net CRYSTAL_1: now also U5.1 (PA00)
- net CRYSTAL_2: now also U5.2 (PA01)
- net D10: now also J8.2, U5.41 (PA20)
- net D11: now also U5.42 (PA21)
- net D12: now also U5.43 (PA22)
- net D13: now also U5.44 (PA23)
- net D4: now also U5.31 (PA14)
- net D5: now also U5.35 (PA16)
- net D6: now also U5.37 (PA18)
- net D8_NEOPIX: now also LED1.3 (DI), U4.4 (BY); no longer LED1.1 (DI)
- net D9: now also U5.38 (PA19)
- net GND: now also LED1.2 (GND), R15.2, SW1.3 (S), SW1.4 (S1), C18.2, C19.2, C20.2, J8.10, J8.13, J8.16, J8.6, J8.S-1 (SHIELD), J8.S-2 (SHIELD__1), J8.S-4 (SHIELD__2), J8.S-5 (SHIELD__3), J8.S-6 (SHIELD__4), U4.2 (GND), U5.22 (GND), U5.33 (GND), U5.47 (GND), U5.54 (GND), U5.65 (EPAD), U5.7 (GND); no longer D3.1 (K), LED1.4 (GND), SW1.B (S), SW1.B' (S1)
- net LDO_INPUT: now also D4.1
- net MCU_SWCLK: now also U5.57 (PA30)
- net MCU_SWDIO: now also U5.58 (PA31)
- net MISO: now also J8.7, U5.49 (PB22)
- net MOSI: now also J8.3, U5.50 (PB23)
- net QSPI_CS: now also U5.24 (PB11)
- net RX_D0: now also U5.40 (PB17)
- net SCK: now also J8.5, U5.36 (PA17)
- net SCL: now also U5.30 (PA13)
- net SDA: now also U5.29 (PA12)
- net TX_D1: now also U5.39 (PB16)
- net USB_D+: now also U5.46 (PA25)
- net USB_D-: now also U5.45 (PA24)
- net VBUS: now also C17.1, LED1.4 (VDD), R2.1, C20.1, D4.2, U4.5 (OE), U4.6 (VCCB); no longer D1.2 (A)
- net ~{RESET}: now also SW1.1 (P), SW1.2 (P1), U5.52 (~{RESETN}); no longer SW1.A (P), SW1.A' (P1)
- net LIPO_STAT: now reaches D1.1 (K)
- net LIPO_STAT: now also D3.2 (A), U3.1 (STAT); no longer R2.1
- net LIPO_PROG: now reaches R8.1, U3.5 (PROG)
- net at C13.1, C15.1, L2.1: now also U5.53 (VDDCORE)
- net at L2.2: now also U5.55 (VSW)
- net at TP1.1: now also LED1.1 (DO); no longer LED1.3 (DO)
- net QSPI_DATA[0] renamed QSPI_DATA_0
- net QSPI_DATA_0: now also U5.17 (PA08)
- net QSPI_DATA[1] renamed QSPI_DATA_1
- net QSPI_DATA_1: now also U5.18 (PA09)
- net QSPI_DATA[2] renamed QSPI_DATA_2
- net QSPI_DATA_2: now also U5.19 (PA10)
- net QSPI_DATA[3] renamed QSPI_DATA_3
- net QSPI_DATA_3: now also U5.20 (PA11)
- net QSPI_SCK renamed QSPI_CLOCK
- net QSPI_CLOCK: now also U5.23 (PB10)
- net V_DIV renamed BATT_VOLT_DIVIDER
- net BATT_VOLT_DIVIDER: now also U5.62 (PB01)
- new net: D1.2 (A), R2.2
- new net: D3.1 (K), R15.1
- new net MCU_D8_NEOPIX: U4.3 (A), U5.64 (PB03)
- no-connect marks 23 -> 29
Other:
- removed sheet SAMD51-BGA
- note added: "3.7V - 4.2V"
- note added: "4.75 to 5.25 V"
- note added: "600 mA Maximum"
- note added: "BATTERY CHARGING R8 = Charge Current 10K = 100mA 5.0K = 200mA 2.0K = 500mA 1.0K = 1000mA"
- note added: "Battery Connector S2B-PH-SM4-TB Side Entry"
- note added: "CAN1_TX CAN1_RX CAN1_TX CAN1_RX"
- note added: "Chip Select Data Input Serial Clock Data Out"
- note added: "LOGIC LEVEL SHIFTER 3V -> 5V Logic"
- note added: "Micro SD Card Holder"
- note added: "NEOPIXEL / SK6812MINI https://www.adafruit.com/product/2659 https://www.adafruit.com/product/2686"
- note added: "NOR Flash W25Q128JVSIQ W25Q64JVSSIQ Previous NOR Flash Memory Part Number: W25Q16JVUXIQ Footprint: USON8 2mm x 3mm"
- note added: "NOTES: Resistors have a 1% tolerance unless stated otherwise. Capacitors have a 10% tolerance unless stated otherwise."
- note added: "PCC: DEN1: SDA DEN2: SCL CLK: D6 D0: D11 D1: D13 D2: D10 D3: D12 D4: MISO D5: D5 D6: MOSI D7: SCK SPI: SERCOM1 DOPO = 0x3, SCK.1 & MO.3, MI.2 I2C: SERCOM2 or 4 UART: SERCOM5, TX on .0 & RX on .1 SPI Flash: QSPI (dual io) Internal SPI on SERCOM 2 I2S: SCK0: A2 FS0: MISO SDI: MOSI SDO: D5 TCC1: WO0: D11 WO1: D13 WO2: D10 WO3: D12 WO4: MISO WO5: D5 WO6: MOSI WO7: SCK"
- note added: "PCCD0 PCCD1 PCCD2 PCCD3 PCCD4 PCCD5 PCCD6 CAN0_TX PCCD7 CAN0_RX"
- note added: "PCCDEN1 PCCDEN2 PCCLK"
- note added: "QWIIC BM04B-SRSS-TB Top Entry SM04B-SRSS-TB Side Entry"
- note added: "USB4105-GF-A"
- note removed: "1.0K = 1000mA"
- note removed: "10K = 100mA"
- note removed: "2.0K = 500mA"
- note removed: "5.0K = 200mA"
- note removed: "Add a SN74AHCT1G125 buffer for the NeoPixel data input and connect the NeoPixel to 5V. Length match the NOR Flash signals? SDHC0 / SDHC1 are available on the TFBGA 120 Package Length match the Micro SD card signals to 50 mil?"
- note removed: "BM04B-SRSS-TB Top Entry SM04B-SRSS-TB Side Entry"
- note removed: "CAN0_RX"
- note removed: "CAN0_TX"
- note removed: "CAN1_RX"
- note removed: "CAN1_TX"
- note removed: "Change the 1 uF 0603 capacitor to a 10 uF 0805? Look for larger X7R capacitors in a 0603 footprint."
- note removed: "PCC: DEN1: SDA DEN2: SCL CLK: D6 D0: D11 D1: D13 D2: D10 D3: D12 D4: MISO D5: D5 D6: MOSI D7: SCK SPI: SERCOM1 DOPO = 0x3, SCK.1 & MO.3, MI.2 I2C: SERCOM2 or 4 UART: SERCOM5, TX on .0 & RX on .1 SPI Flash: QSPI (dual io) I2S: SCK0: A2 FS0: MISO SDI: MOSI SDO: D5 TCC1: WO0: D11 WO1: D13 WO2: D10 WO3: D12 WO4: MISO WO5: D5 WO6: MOSI WO7: SCK"
- note removed: "PCCD0"
- note removed: "PCCD1"
- note removed: "PCCD2"
- note removed: "PCCD3"
- note removed: "PCCD4"
- note removed: "PCCD5"
- note removed: "PCCD6"
- note removed: "PCCD7"
- note removed: "PCCDEN1"
- note removed: "PCCDEN2"
- note removed: "PCCLK"
- note removed: "POWER AND FILTERING"
- note removed: "RED LED"
- note removed: "S2B-PH-SM4-TB"
- note removed: "USB AND BATTERY CHARGING"
- note removed: "W25Q128JVSIQ W25Q64JVSSIQ Previous Flash Memory Part Number: W25Q16JVUXIQ Footprint: USON8 2mm x 3mm"
- note removed: "https://www.adafruit.com/product/2659 https://www.adafruit.com/product/2686"
- moved on the sheet: C14, C16, C17, C2, C3, C4, C6, C8, J1, J3, J4, J5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
